File: desainPCB/concentrator.sch (EAGLE design)
At the start: 23 parts, among them M1 ARDUINO-PRO-MINI-5.0V, M2 ARDUINO-PRO-MINI-5.0V, M3 ARDUINO-PRO-MINI-5.0V, M4 ARDUINO-PRO-MINI-5.0V

Commit message: new sensor suhu
Parts:
- removed D1: 1N5060GP, diode:1N5060GP
- added KANAN4, KANAN5, KIRI4, KIRI5: (no value), pinhead:PINHD-1X8
- added KANANFT4, KANANFT5, KIRIFT4, KIRIFT5: (no value), pinhead:PINHD-1X9
- added M5, M6: ARDUINO-PRO-MINI-5.0V, diy-modules:ARDUINO-PRO-MINI-5.0V
Connections:
- removed net 10: KANAN.2, KANAN1.2, KANAN2.2, KANAN3.2, M1.D10, M2.D10, M3.D10, M4.D10
- removed net 11: KANAN.3, KANAN1.3, KANAN2.3, KANAN3.3, M1.D11, M2.D11, M3.D11, M4.D11
- removed net 12: KANAN.4, KANAN1.4, KANAN2.4, KANAN3.4, M1.D12, M2.D12, M3.D12, M4.D12
- removed net 13: KANAN.5, KANAN1.5, KANAN2.5, KANAN3.5, M1.D13, M2.D13, M3.D13, M4.D13
- removed net 2: KIRI.5, KIRI1.5, KIRI2.5, KIRI3.5, M1.D2, M2.D2, M3.D2, M4.D2
- removed net 4: M2.D4
- removed net 9: KIRI.4, KIRI1.4, KIRI2.4, KIRI3.4, M1.D9, M2.D9, M3.D9, M4.D9
- removed net D3: M4.D3
- removed net GND: 12V-5V1.IN-, 12V-5V1.OUT-, KIRI.1, KIRI.2, KIRI1.1, KIRI1.2, KIRI2.1, KIRI2.2, KIRI3.1, KIRI3.2, KIRIFT.3, KIRIFT1.3, KIRIFT2.3, KIRIFT3.3, M1.GND.2, M2.GND.2, M3.GND.2, M4.GND.2, U$1.P0
- removed net N$1: 12V-5V1.IN+, D1.C
- removed net N$2: D1.A, U$1.P1
- removed net RXD: KIRIFT.5, KIRIFT1.5, KIRIFT2.5, KIRIFT3.5, M1.D1/TX, M2.D1/TX, M3.D1/TX, M4.D1/TX
- removed net TXD: KIRIFT.9, KIRIFT1.9, KIRIFT2.9, KIRIFT3.9, M1.D0/RX, M2.D0/RX, M3.D0/RX, M4.D0/RX
- new net 10.1: KANAN.2, M1.D10
- new net 10.2: KANAN2.2, M3.D10
- new net 10.3: KANAN1.2, M2.D10
- new net 10.4: KANAN3.2, M4.D10
- new net 10.5: KANAN4.2, M5.D10
- new net 10.6: KANAN5.2, M6.D10
- new net 11.1: KANAN.3, M1.D11
- new net 11.2: KANAN2.3, M3.D11
- new net 11.3: KANAN1.3, M2.D11
- new net 11.4: KANAN3.3, M4.D11
- new net 11.5: KANAN4.3, M5.D11
- new net 11.6: KANAN5.3, M6.D11
- new net 12.1: KANAN.4, M1.D12
- new net 12.2: KANAN2.4, M3.D12
- new net 12.3: KANAN1.4, M2.D12
- new net 12.4: KANAN3.4, M4.D12
- new net 12.5: KANAN4.4, M5.D12
- new net 12.6: KANAN5.4, M6.D12
- new net 13.1: KANAN.5, M1.D13
- new net 13.2: KANAN2.5, M3.D13
- new net 13.3: KANAN1.5, M2.D13
- new net 13.4: KANAN3.5, M4.D13
- new net 13.5: KANAN4.5, M5.D13
- new net 13.6: KANAN5.5, M6.D13
- new net 2.1: KIRI.5, M1.D2
- new net 2.2: KIRI2.5, M3.D2
- new net 2.3: KIRI1.5, M2.D2
- new net 2.4: KIRI3.5, M4.D2
- new net 2.5: KIRI4.5, M5.D2
- new net 2.6: KIRI5.5, M6.D2
- new net 4.5: M5.D4
- new net 8.5: M5.D8
- new net 9.1: KIRI.4, M1.D9
- new net 9.2: KIRI2.4, M3.D9
- new net 9.3: KIRI1.4, M2.D9
- new net 9.4: KIRI3.4, M4.D9
- new net 9.5: KIRI4.4, M5.D9
- new net 9.6: KIRI5.4, M6.D9
- new net GND.1: 12V-5V1.IN-, 12V-5V1.OUT-, KIRI.1, KIRI.2, KIRI1.1, KIRI1.2, KIRI2.1, KIRI2.2, KIRI3.1, KIRI3.2, KIRI4.1, KIRI4.2, KIRI5.1, KIRI5.2, KIRIFT.3, KIRIFT1.3, KIRIFT2.3, KIRIFT3.3, KIRIFT4.3, KIRIFT5.3, M1.GND.2, M2.GND.2, M3.GND.2, M4.GND.2, M5.GND.2, M6.GND.2, U$1.P0
- new net IN+: U$1.P1
- new net OUT+: 12V-5V1.IN+
- new net RXD.1: KIRIFT2.5, M1.D1/TX
- new net RXD.2: KIRIFT1.5, M3.D1/TX
- new net RXD.3: KIRIFT3.5, M2.D1/TX
- new net RXD.4: KIRIFT.5, M4.D1/TX
- new net RXD.5: KIRIFT4.5, M5.D1/TX
- new net RXD6: KIRIFT5.5, M6.D1/TX
- new net TXD.1: KIRIFT2.9, M1.D0/RX
- new net TXD.2: KIRIFT1.9, M3.D0/RX
- new net TXD.3: KIRIFT3.9, M2.D0/RX
- new net TXD.4: KIRIFT.9, M4.D0/RX
- new net TXD.5: KIRIFT4.9, M5.D0/RX
- new net TXD6: KIRIFT5.9, M6.D0/RX
- net 3V: now also KIRI4.3, KIRI5.3, KIRIFT4.6, KIRIFT5.6, M5.VCC, M6.VCC
- net 8: no longer M2.D8
Other:
- moved on the sheet: KANAN1, KANAN3, KANANFT, KANANFT3, KIRI1, KIRI3, KIRIFT, KIRIFT3, M2, M4
