File: desainPCB/rtu04_full bridge.brd (EAGLE design)
At the start: 78.7 x 77.1 mm, 17 parts, among them M1 ARDUINO-PRO-MINI-5.0V, X1 JST-XH-02-PIN-LONG-PAD

Commit message: desain baru pcb
Parts:
- removed R1, R2, R3: (no value), rcl:0207/10
- added U$4, U$5, U$6: DBCONN-1X2, Terminal Block Connector:DBCONN-1X2
Connections:
- net A+: now also U$4.P1; no longer R2.2
- net A-: now also U$5.P0, U$6.P1; no longer R1.1, R3.1
- net E+: now also U$4.P0, U$5.P1; no longer R1.2, R2.1
- net E-: now also U$6.P0; no longer R3.2
Routing:
- net E+: track 39.2 -> 66.1 mm, vias 0 -> 1
- net E-: track 38.6 -> 56.8 mm
- net A2: track 76.2 -> 66.0 mm
- net A+: track 45.9 -> 50.7 mm, vias 0 -> 1
- net A-: track 28.1 -> 26.4 mm
Changed lines of the file:
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@@
 <layer number="43" name="vRestrict" color="2" fill="10" visible="yes" active="yes"/>
 <layer number="44" name="Drills" color="7" fill="1" visible="no" active="yes"/>
-<layer number="45" name="Holes" color="7" fill="1" visible="no" active="yes"/>
+<layer number="45" name="Holes" color="7" fill="1" visible="yes" active="yes"/>
 <layer number="46" name="Milling" color="3" fill="1" visible="no" active="yes"/>
 <layer number="47" name="Measures" color="7" fill="1" visible="no" active="yes"/>
@@
 <hole x="71.12" y="72.39" drill="3"/>
 <hole x="55.88" y="12.7" drill="3"/>
-<hole x="3.81" y="60.96" drill="3"/>
+<hole x="5.08" y="60.96" drill="3"/>
 <text x="5.08" y="30.48" size="1.778" layer="21">+</text>
 <text x="13.97" y="59.69" size="1.778" layer="21">+</text>
@@
 </element>
 <element name="U$2" library="Terminal Block Connector" package="DBCONN-1X2" value="DBCONN-1X2" x="5.08" y="71.12" smashed="yes" rot="R270"/>
-<element name="R1" library="rcl" library_urn="urn:adsk.eagle:library:334" package="0207/10" package3d_urn="urn:adsk.eagle:package:23491/2" value="" x="34.29" y="71.12" smashed="yes">
-<attribute name="NAME" x="31.242" y="72.644" size="1.27" layer="25" ratio="10"/>
-<attribute name="POPULARITY" value="81" x="34.29" y="71.12" size="1.778" layer="27" display="off"/>
-<attribute name="SPICEPREFIX" value="R" x="34.29" y="71.12" size="1.778" layer="27" display="off"/>
-<attribute name="VALUE" x="32.0294" y="70.485" size="1.27" layer="27" ratio="10"/>
-</element>
-<element name="R2" library="rcl" library_urn="urn:adsk.eagle:library:334" package="0207/10" package3d_urn="urn:adsk.eagle:package:23491/2" value="" x="20.32" y="73.66" smashed="yes" rot="R180">
-<attribute name="NAME" x="23.368" y="72.136" size="1.27" layer="25" ratio="10" rot="R180"/>
-<attribute name="POPULARITY" value="81" x="20.32" y="73.66" size="1.778" layer="27" rot="R180" display="off"/>
-<attribute name="SPICEPREFIX" value="R" x="20.32" y="73.66" size="1.778" layer="27" rot="R180" display="off"/>
-<attribute name="VALUE" x="22.5806" y="74.295" size="1.27" layer="27" ratio="10" rot="R180"/>
-</element>
-<element name="R3" library="rcl" library_urn="urn:adsk.eagle:library:334" package="0207/10" package3d_urn="urn:adsk.eagle:package:23491/2" value="" x="20.32" y="68.58" smashed="yes" rot="R180">
-<attribute name="NAME" x="23.368" y="67.056" size="1.27" layer="25" ratio="10" rot="R180"/>
-<attribute name="POPULARITY" value="81" x="20.32" y="68.58" size="1.778" layer="27" rot="R180" display="off"/>
-<attribute name="SPICEPREFIX" value="R" x="20.32" y="68.58" size="1.778" layer="27" rot="R180" display="off"/>
-<attribute name="VALUE" x="22.5806" y="69.215" size="1.27" layer="27" ratio="10" rot="R180"/>
-</element>
 <element name="U$3" library="diy-modules (1)" package="BATTERY-CHARGER-LI-5V" value="BATTERY-CHARGER-LI-5V" x="15.24" y="12.7" smashed="yes">
 <attribute name="NAME" x="15.24" y="24.13" size="1.27" layer="25" align="bottom-center"/>
@@
 <attribute name="VALUE" x="40.005" y="48.26" size="1.27" layer="27" rot="R90"/>
 </element>
+<element name="U$4" library="Terminal Block Connector" package="DBCONN-1X2" value="DBCONN-1X2" x="20.32" y="72.39" smashed="yes"/>
+<element name="U$5" library="Terminal Block Connector" package="DBCONN-1X2" value="DBCONN-1X2" x="43.18" y="72.39" smashed="yes"/>
+<element name="U$6" library="Terminal Block Connector" package="DBCONN-1X2" value="DBCONN-1X2" x="31.75" y="72.39" smashed="yes"/>
 </elements>
 <signals>
@@
 </signal>
 <signal name="E+">
-<contactref element="R1" pad="2"/>
-<contactref element="R2" pad="1"/>
-<wire x1="25.4" y1="73.66" x2="39.37" y2="73.66" width="0.508" layer="16"/>
-<wire x1="39.37" y1="73.66" x2="39.37" y2="71.12" width="0.508" layer="16"/>
 <contactref element="RIGHT" pad="1"/>
-<wire x1="39.37" y1="52.07" x2="36.83" y2="49.53" width="0.508" layer="16"/>
-<wire x1="39.37" y1="71.12" x2="39.37" y2="52.07" width="0.508" layer="16"/>
+<wire x1="36.83" y1="49.53" x2="39.37" y2="52.07" width="0.508" layer="16"/>
+<contactref element="U$4" pad="P0"/>
+<wire x1="17.78" y1="72.39" x2="17.78" y2="69.85" width="0.508" layer="1"/>
+<wire x1="17.78" y1="69.85" x2="25.4" y2="69.85" width="0.508" layer="1"/>
+<wire x1="25.4" y1="69.85" x2="25.4" y2="74.93" width="0.508" layer="1"/>
+<wire x1="25.4" y1="74.93" x2="34.29" y2="74.93" width="0.508" layer="1"/>
+<contactref element="U$5" pad="P1"/>
+<wire x1="34.29" y1="74.93" x2="35.56" y2="74.93" width="0.508" layer="1"/>
+<wire x1="39.37" y1="52.07" x2="39.37" y2="66.04" width="0.508" layer="16"/>
+<via x="39.37" y="66.04" extent="1-16" drill="0.55"/>
+<wire x1="39.37" y1="66.04" x2="40.64" y2="67.31" width="0.508" layer="1"/>
+<wire x1="40.64" y1="67.31" x2="45.72" y2="67.31" width="0.508" layer="1"/>
+<wire x1="45.72" y1="67.31" x2="45.72" y2="72.31" width="0.508" layer="1"/>
+<wire x1="45.72" y1="72.31" x2="45.64" y2="72.39" width="0.508" layer="1"/>
+<wire x1="35.56" y1="74.93" x2="43.1" y2="74.93" width="0.508" layer="1"/>
+<wire x1="43.1" y1="74.93" x2="45.64" y2="72.39" width="0.508" layer="1"/>
 </signal>
 <signal name="E-">
-<contactref element="R3" pad="2"/>
 <contactref element="U$2" pad="P1"/>
-<wire x1="5.08" y1="68.66" x2="5.16" y2="68.58" width="0.508" layer="16"/>
-<wire x1="5.16" y1="68.58" x2="15.24" y2="68.58" width="0.508" layer="16"/>
 <contactref element="RIGHT" pad="2"/>
-<wire x1="15.24" y1="68.58" x2="31.75" y2="52.07" width="0.508" layer="16"/>
-<wire x1="31.75" y1="52.07" x2="36.83" y2="52.07" width="0.508" layer="16"/>
+<wire x1="29.21" y1="52.07" x2="36.83" y2="52.07" width="0.508" layer="16"/>
+<contactref element="U$6" pad="P0"/>
+<wire x1="5.08" y1="68.66" x2="8.97" y2="64.77" width="0.508" layer="16"/>
+<wire x1="29.21" y1="72.39" x2="29.21" y2="52.07" width="0.508" layer="16"/>
+<wire x1="21.59" y1="64.77" x2="29.21" y2="72.39" width="0.508" layer="16"/>
+<wire x1="8.97" y1="64.77" x2="21.59" y2="64.77" width="0.508" layer="16"/>
 </signal>
 <signal name="A-">
-<contactref element="R3" pad="1"/>
-<contactref element="R1" pad="1"/>
-<wire x1="29.21" y1="71.12" x2="26.67" y2="68.58" width="0.508" layer="16"/>
-<wire x1="25.4" y1="68.58" x2="26.67" y2="68.58" width="0.508" layer="16"/>
-<wire x1="25.4" y1="68.58" x2="33.02" y2="68.58" width="0.508" layer="16"/>
-<wire x1="33.02" y1="68.58" x2="33.02" y2="58.22" width="0.508" layer="16"/>
 <contactref element="RIGHT" pad="3"/>
-<wire x1="33.02" y1="58.22" x2="36.63" y2="54.61" width="0.508" layer="16"/>
+<wire x1="36.63" y1="54.61" x2="33.02" y2="58.22" width="0.508" layer="16"/>
 <wire x1="36.63" y1="54.61" x2="36.83" y2="54.61" width="0.508" layer="16"/>
+<contactref element="U$6" pad="P1"/>
+<contactref element="U$5" pad="P0"/>
+<wire x1="33.02" y1="71.2" x2="34.21" y2="72.39" width="0.508" layer="16"/>
+<wire x1="33.02" y1="58.22" x2="33.02" y2="71.2" width="0.508" layer="16"/>
+<wire x1="34.21" y1="72.39" x2="40.64" y2="72.39" width="0.508" layer="16"/>
 </signal>
 <signal name="A+">
-<contactref element="R2" pad="2"/>
 <contactref element="U$2" pad="P0"/>
-<wire x1="5.08" y1="73.66" x2="15.24" y2="73.66" width="0.508" layer="16"/>
-<wire x1="15.24" y1="73.66" x2="13.97" y2="72.39" width="0.508" layer="1"/>
-<wire x1="13.97" y1="72.39" x2="12.7" y2="72.39" width="0.508" layer="1"/>
-<wire x1="12.7" y1="72.39" x2="12.7" y2="68.58" width="0.508" layer="1"/>
-<wire x1="12.7" y1="68.58" x2="20.32" y2="60.96" width="0.508" layer="1"/>
-<wire x1="20.32" y1="60.96" x2="31.75" y2="60.96" width="0.508" layer="1"/>
+<wire x1="20.32" y1="60.96" x2="33.02" y2="60.96" width="0.508" layer="1"/>
 <contactref element="RIGHT" pad="4"/>
-<wire x1="31.75" y1="60.96" x2="32.82" y2="60.96" width="0.508" layer="1"/>
-<wire x1="32.82" y1="60.96" x2="33.02" y2="60.96" width="0.508" layer="1"/>
 <wire x1="33.02" y1="60.96" x2="36.83" y2="57.15" width="0.508" layer="1"/>
+<contactref element="U$4" pad="P1"/>
+<wire x1="22.86" y1="72.39" x2="22.78" y2="72.39" width="0.508" layer="1"/>
+<wire x1="5.08" y1="73.66" x2="6.35" y2="74.93" width="0.508" layer="1"/>
+<wire x1="6.35" y1="74.93" x2="21.59" y2="74.93" width="0.508" layer="1"/>
+<wire x1="21.59" y1="74.93" x2="22.86" y2="73.66" width="0.508" layer="1"/>
+<wire x1="22.86" y1="73.66" x2="22.86" y2="72.39" width="0.508" layer="1"/>
+<via x="20.32" y="67.31" extent="1-16" drill="0.55"/>
+<wire x1="20.32" y1="67.31" x2="20.32" y2="60.96" width="0.508" layer="1"/>
+<wire x1="22.78" y1="72.39" x2="22.78" y2="69.77" width="0.508" layer="16"/>
+<wire x1="22.78" y1="69.77" x2="20.32" y2="67.31" width="0.508" layer="16"/>
 </signal>
 <signal name="A1">
@@
 <contactref element="LEFT" pad="3"/>
 <wire x1="40.64" y1="60.96" x2="40.64" y2="64.77" width="0.508" layer="1"/>
-<wire x1="40.64" y1="64.77" x2="22.86" y2="64.77" width="0.508" layer="1"/>
-<wire x1="22.86" y1="64.77" x2="22.86" y2="63.5" width="0.508" layer="1"/>
-<wire x1="22.86" y1="63.5" x2="25.4" y2="63.5" width="0.508" layer="1"/>
-<wire x1="25.4" y1="63.5" x2="25.4" y2="62.23" width="0.508" layer="1"/>
-<via x="25.4" y="62.23" extent="1-16" drill="0.55"/>
-<wire x1="25.4" y1="62.23" x2="25.4" y2="59.69" width="0.508" layer="16"/>
-<wire x1="25.4" y1="59.69" x2="27.94" y2="59.69" width="0.508" layer="16"/>
-<via x="27.94" y="59.69" extent="1-16" drill="0.55"/>
-<wire x1="27.94" y1="59.69" x2="27.94" y2="57.15" width="0.508" layer="1"/>
+<wire x1="40.64" y1="64.77" x2="27.94" y2="64.77" width="0.508" layer="1"/>
+<via x="27.94" y="64.77" extent="1-16" drill="0.55"/>
+<wire x1="27.94" y1="64.77" x2="27.94" y2="58.42" width="0.508" layer="16"/>
+<via x="27.94" y="58.42" extent="1-16" drill="0.55"/>
+<wire x1="27.94" y1="58.42" x2="27.94" y2="57.15" width="0.508" layer="1"/>
 <wire x1="27.94" y1="57.15" x2="16.51" y2="57.15" width="0.508" layer="1"/>
 </signal>
